File: Generic Toolhead.kicad_sch (KiCad schematic)
At the start: 23 parts

Commit message: Update Generic Toolhead.kicad_sch
Other:
- note added: "24V in. USB in. Permanent ADXL345. Permanent TMC2209. Heater (or multiple?) Thermistor (or multiple?) Fans. Read EEPROM. Speakers. Is there some way to make some of those genericy?"
- note removed: "24V in. USB in. Permanent ADXL345. Permanent TMC2209. Heater (or multiple?) Thermistor (or multiple?) Fans. Is there some way to make some of those genericy?"
Changed lines of the file:
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@@
     (effects (font (size 1.27 1.27)) (justify left bottom))
   )
-  (text "24V in.\nUSB in.\n\nPermanent ADXL345.\nPermanent TMC2209.\nHeater (or multiple?)\nThermistor (or multiple?)\nFans.\n\nIs there some way to make some of those genericy?"
+  (text "24V in.\nUSB in.\n\nPermanent ADXL345.\nPermanent TMC2209.\nHeater (or multiple?)\nThermistor (or multiple?)\nFans.\nRead EEPROM.\nSpeakers.\n\nIs there some way to make some of those genericy?"
     (at 13.97 195.58 0)
     (effects (font (size 1.27 1.27)) (justify left bottom))

Commit message: .
Parts:
- added C?: 1u, symbol Device:C_Small
- added C?: 0u1, symbol Device:C_Small
Connections:
- net +3V3: now also U?.1 (VDD_IO), U?.6 (VS), C?.1, C?.1
- net GND: now also U?.2 (GND), U?.4 (GND), U?.5 (GND), C?.2, C?.2
- net MCU_ADXL_SDO: now reaches U?.12 (SDO)
- net MCU_ADXL_SDA: now reaches U?.13 (SDA)
- net MCU_ADXL_SCL: now reaches U?.14 (SCL)
- net MCU_ADXL_CS: now reaches U?.7 (NCS)
- net MCU_ADXL_INT1: now reaches U?.8 (INT1)
- net MCU_ADXL_INT2: now reaches U?.9 (INT2)
Other:
- moved on the sheet: U?

Commit message: Forgot these bits.
Parts:
- removed C?: 0u1, symbol Device:C_Small
- removed D? (x3): D_Small, symbol Device:D_Small
- removed D?: D_TVS, symbol Device:D_TVS
- removed D?: LED, symbol Device:LED
- removed J? (x2): Conn_01x02_Male, symbol Connector:Conn_01x02_Male
- removed Q?: BUK7M6R3-40EX, Package_TO_SOT_SMD:LFPAK33, symbol Transistor_FET:BUK7M6R3-40EX
- removed R?: 100k, symbol Device:R_Small
- removed R? (x2): 2k37, symbol Device:R_Small
- removed R?: 10, symbol Device:R_Small
- removed R?: 4k7, symbol Device:R_Small
- removed R?: R_Small, symbol Device:R_Small
- removed U?: TMC2209, Package_DFN_QFN:QFN-28-1EP_5x5mm_P0.5mm_EP3.75x3.75mm_ThermalVias, symbol Custom:TMC2209
- C1, C2, C3: renamed from C?; footprint (none) -> Capacitor_SMD:C_0603_1608Metric_Pad1.08x0.95mm_HandSolder
- R1: renamed from R?; footprint (none) -> Resistor_SMD:R_0603_1608Metric_Pad0.98x0.95mm_HandSolder
- gave numbers to parts that had none: 5
Connections:
- net MCU_ADXL_CS: now also U2.18 (GPIO15)
- net MCU_ADXL_SCL: now also U2.15 (GPIO12)
- net MCU_ADXL_SDA: now also U2.16 (GPIO13)
- net MCU_ADXL_SDO: now also U2.17 (GPIO14)
- net Motor Driver/DIR: now reaches U2.2 (GPIO0)
- net Motor Driver/STEP: now reaches U2.3 (GPIO1)
- net Thermistor3/TH_MCU: now reaches U2.38 (GPIO26_ADC0)
- net Thermistor2/TH_MCU: now reaches U2.39 (GPIO27_ADC1)
- net Motor Driver/UART: now reaches U2.4 (GPIO2)
- net Thermistor1/TH_MCU: now reaches U2.40 (GPIO28_ADC2)
- net Thermistor/TH_MCU: now reaches U2.41 (GPIO29_ADC3)
- net MOSFET Driver/INPUT: now reaches U2.5 (GPIO3)
- net MOSFET Driver1/INPUT: now reaches U2.6 (GPIO4)
- net MOSFET Driver2/INPUT: now reaches U2.7 (GPIO5)
- net MOSFET Driver3/INPUT: now reaches U2.8 (GPIO6)
Other:
- added sheet MOSFET Driver (MOSFET Driver.kicad_sch)
- added sheet MOSFET Driver1 (MOSFET Driver.kicad_sch)
- added sheet MOSFET Driver2 (MOSFET Driver.kicad_sch)
- added sheet MOSFET Driver3 (MOSFET Driver.kicad_sch)
- added sheet Motor Driver (Motor Driver.kicad_sch)
- added sheet Thermistor (Thermistor.kicad_sch)
- added sheet Thermistor1 (Thermistor.kicad_sch)
- added sheet Thermistor2 (Thermistor.kicad_sch)
- added sheet Thermistor3 (Thermistor.kicad_sch)
- note removed: "MOSFET is chosen at random. Not actual part. This circuit is for both heaters and fans, just different mosfets. MOS_MCU should be run through a buffer gate/voltage converter."
- note removed: "Thermistor circuit from BTT SKR Mini E3V3"
- moved on the sheet: C2, C3, U1, U2

Commit message: More big changes. Almost entirely done.
Parts:
- removed C2: 0u1, Capacitor_SMD:C_0603_1608Metric_Pad1.08x0.95mm_HandSolder, symbol Device:C_Small
- removed C3: 1u, Capacitor_SMD:C_0603_1608Metric_Pad1.08x0.95mm_HandSolder, symbol Device:C_Small
- removed U1: ADXL345, Package_LGA:LGA-14_3x5mm_P0.8mm_LayoutBorder1x6y, symbol Custom:ADXL345
- added C15, C19, C21, C23, C25, C28: 100n, Capacitor_SMD:C_0603_1608Metric_Pad1.08x0.95mm_HandSolder, symbol Device:C_Small
- added C16, C18, C22, C24: 100n, Capacitor_SMD:C_0402_1005Metric_Pad0.74x0.62mm_HandSolder, symbol Device:C_Small
- added C17, C20: 1u, Capacitor_SMD:C_0402_1005Metric_Pad0.74x0.62mm_HandSolder, symbol Device:C_Small
- added C26, C27: 10u, Capacitor_SMD:C_0603_1608Metric_Pad1.08x0.95mm_HandSolder, symbol Device:C_Small
- added R24, R25: 27_4, Resistor_SMD:R_0402_1005Metric_Pad0.72x0.64mm_HandSolder, symbol Device:R_Small
- added R26: 1k, Resistor_SMD:R_0603_1608Metric_Pad0.98x0.95mm_HandSolder, symbol Device:R_Small
- added R27: 10k, Resistor_SMD:R_0603_1608Metric_Pad0.98x0.95mm_HandSolder, symbol Device:R_Small
- added SW1: SW_DIP_x01, symbol Switch:SW_DIP_x01
- added U4: AP1117-33, Package_TO_SOT_SMD:SOT-223-3_TabPin2, symbol Regulator_Linear:AP1117-33
- added U5: W25Q128JVS, Package_SO:SOIC-8_5.23x5.23mm_P1.27mm, symbol Memory_Flash:W25Q128JVS
- J2: footprint (none) -> Connector_USB:USB_C_Receptacle_HRO_TYPE-C-31-M-12
Connections:
- net +3V3: now also U2.1 (IOVDD), U2.10 (IOVDD), U2.22 (IOVDD), U2.33 (IOVDD), U2.42 (IOVDD), U2.43 (ADC_AVDD), U2.44 (VREG_IN), U2.48 (USB_VDD), U2.49 (IOVDD), C18.1, C19.1, C20.1, C21.1, C22.1, C23.1, C24.1, C25.1, C27.1, C28.1, R27.1, U4.2 (VO), U5.8 (VCC)
- net GND: now also C15.2, C16.2, C17.2, C18.2, C19.2, C20.2, C21.2, C22.2, C23.2, C24.2, C25.2, C26.2, C27.2, C28.2, SW1.1, U4.1 (GND)
- net USB_DM: now also R25.2; no longer U2.46 (USB_DM)
- net USB_DP: now also R24.1; no longer U2.47 (USB_DP)
- net Oscillator/XIN: now reaches U2.20 (XIN)
- net Oscillator/XOUT: now reaches U2.21 (XOUT)
- net +1V1: now reaches U2.23 (DVDD), U2.50 (DVDD)
- net +1V1: now also U2.45 (VREG_VOUT), C15.1, C16.1, C17.1
- net QSPI_SD3: now reaches U2.51 (QSPI_SD3)
- net QSPI_SD3: now also U5.7 (IO3)
- net QSPI_SCLK: now reaches U2.52 (QSPI_SCLK)
- net QSPI_SCLK: now also U5.6 (CLK)
- net QSPI_SD0: now reaches U2.53 (QSPI_SD0)
- net QSPI_SD0: now also U5.5 (DI(IO0))
- net QSPI_SD2: now reaches U2.54 (QSPI_SD2)
- net QSPI_SD2: now also U5.3 (IO2)
- net QSPI_SD1: now reaches U2.55 (QSPI_SD1)
- net QSPI_SD1: now also U5.2 (DO(IO1))
- net QSPI_SS: now reaches U2.56 (QSPI_SS)
- net QSPI_SS: now also R26.2, R27.2, U5.1 (~{CS})
- net VBUS: now reaches J2.A4 (VBUS), J2.A9 (VBUS), J2.B4 (VBUS), J2.B9 (VBUS)
- net VBUS: now also C26.1, U4.3 (VI)
- net MCU_ADXL_CS renamed ADXL/CS
- net MCU_ADXL_SCL renamed ADXL/SCL
- net MCU_ADXL_SDA renamed ADXL/SDA
- net MCU_ADXL_SDO renamed ADXL/SDO
- new net: R24.2, U2.47 (USB_DP)
- new net: R26.1, SW1.2
- new net: R25.1, U2.46 (USB_DM)
Other:
- added sheet ADXL (ADXL.kicad_sch)
- added sheet Oscillator (Oscillator.kicad_sch)
- note added: "Read EEPROM. Speakers. Is there some way to make some of those genericly?"
- note removed: "24V in. USB in. Permanent ADXL345. Permanent TMC2209. Heater (or multiple?) Thermistor (or multiple?) Fans. Read EEPROM. Speakers. Is there some way to make some of those genericy?"
- note removed: "Do I need resistors for the USB stuff? I think so, I should do that."
- moved on the sheet: D1
