File: MOSFET Driver.kicad_sch (KiCad schematic)
At the start: 6 parts, among them Q1 LND150

Commit message: More big changes. Almost entirely done.
Parts:
- renumbered D14 to D17, Q1 to Q4, R16 to R22, R17 to R23, TP9 to TP15, TP10 to TP16
Changed lines of the file:
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@@
   (symbol (lib_id "Connector:TestPoint") (at 118.745 33.02 270) (unit 1)
     (in_bom yes) (on_board yes)
-    (property "Reference" "TP10" (id 0) (at 124.46 33.02 90)
+    (property "Reference" "TP16" (id 0) (at 124.46 33.02 90)
       (effects (font (size 1.27 1.27)) (justify left))
     )
@@
   (symbol (lib_id "power:GND") (at 99.06 50.8 0) (unit 1)
     (in_bom yes) (on_board yes) (fields_autoplaced)
-    (property "Reference" "#PWR039" (id 0) (at 99.06 57.15 0)
+    (property "Reference" "#PWR0105" (id 0) (at 99.06 57.15 0)
       (effects (font (size 1.27 1.27)) hide)
     )
@@
   (symbol (lib_id "Device:D_Small") (at 99.06 25.4 270) (unit 1)
     (in_bom yes) (on_board yes) (fields_autoplaced)
-    (property "Reference" "D14" (id 0) (at 101.6 24.1299 90)
+    (property "Reference" "D17" (id 0) (at 101.6 24.1299 90)
       (effects (font (size 1.27 1.27)) (justify left))
     )
@@
   (symbol (lib_id "power:GND") (at 118.745 33.02 0) (unit 1)
     (in_bom yes) (on_board yes) (fields_autoplaced)
-    (property "Reference" "#PWR0101" (id 0) (at 118.745 39.37 0)
+    (property "Reference" "#PWR0107" (id 0) (at 118.745 39.37 0)
       (effects (font (size 1.27 1.27)) hide)
     )
@@
   (symbol (lib_id "Device:R_Small") (at 81.28 38.1 90) (unit 1)
     (in_bom yes) (on_board yes) (fields_autoplaced)
-    (property "Reference" "R16" (id 0) (at 81.28 31.75 90))
+    (property "Reference" "R22" (id 0) (at 81.28 31.75 90))
     (property "Value" "10" (id 1) (at 81.28 34.29 90))
     (property "Footprint" "Resistor_SMD:R_0603_1608Metric_Pad0.98x0.95mm_HandSolder" (id 2) (at 81.28 38.1 0)
@@
   (symbol (lib_id "Device:R_Small") (at 87.63 45.72 180) (unit 1)
     (in_bom yes) (on_board yes) (fields_autoplaced)
-    (property "Reference" "R17" (id 0) (at 90.17 44.4499 0)
+    (property "Reference" "R23" (id 0) (at 90.17 44.4499 0)
       (effects (font (size 1.27 1.27)) (justify right))
     )
@@
   (symbol (lib_id "Connector:TestPoint") (at 118.745 30.48 270) (unit 1)
     (in_bom yes) (on_board yes)
-    (property "Reference" "TP9" (id 0) (at 124.46 30.48 90)
+    (property "Reference" "TP15" (id 0) (at 124.46 30.48 90)
       (effects (font (size 1.27 1.27)) (justify left))
     )
@@
   (symbol (lib_id "power:GND") (at 87.63 50.8 0) (unit 1)
     (in_bom yes) (on_board yes) (fields_autoplaced)
-    (property "Reference" "#PWR038" (id 0) (at 87.63 57.15 0)
+    (property "Reference" "#PWR0106" (id 0) (at 87.63 57.15 0)
       (effects (font (size 1.27 1.27)) hide)
     )
@@
   (symbol (lib_id "Device:Q_NMOS_GDS") (at 96.52 38.1 0) (unit 1)
     (in_bom yes) (on_board yes) (fields_autoplaced)
-    (property "Reference" "Q1" (id 0) (at 102.87 36.8299 0)
+    (property "Reference" "Q4" (id 0) (at 102.87 36.8299 0)
       (effects (font (size 1.27 1.27)) (justify left))
     )

Commit message: Far better layout.
Parts:
- TP15, TP16: footprint TestPoint:TestPoint_THTPad_2.5x2.5mm_Drill1.2mm -> Library:Pogo Pin
Changed lines of the file:
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@@
       (effects (font (size 1.27 1.27)) (justify left) hide)
     )
-    (property "Footprint" "TestPoint:TestPoint_THTPad_2.5x2.5mm_Drill1.2mm" (id 2) (at 118.745 38.1 0)
+    (property "Footprint" "Library:Pogo Pin" (id 2) (at 118.745 38.1 0)
       (effects (font (size 1.27 1.27)) hide)
     )
@@
       (effects (font (size 1.27 1.27)) (justify left) hide)
     )
-    (property "Footprint" "TestPoint:TestPoint_THTPad_2.5x2.5mm_Drill1.2mm" (id 2) (at 118.745 35.56 0)
+    (property "Footprint" "Library:Pogo Pin" (id 2) (at 118.745 35.56 0)
       (effects (font (size 1.27 1.27)) hide)
     )
