File: Thermistor.kicad_sch (KiCad schematic)
At the start: 9 parts

Commit message: More big changes. Almost entirely done.
Parts:
- renumbered C11 to C12, D2 to D5, D3 to D6, D4 to D7, R4 to R7, R5 to R8, R6 to R9, TP2 to TP4
Changed lines of the file:
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@@
   (symbol (lib_id "Device:R_Small") (at 99.06 39.37 270) (unit 1)
     (in_bom yes) (on_board yes)
-    (property "Reference" "R5" (id 0) (at 99.06 41.91 90))
+    (property "Reference" "R8" (id 0) (at 99.06 41.91 90))
     (property "Value" "2k37" (id 1) (at 99.06 44.45 90))
     (property "Footprint" "Resistor_SMD:R_0603_1608Metric_Pad0.98x0.95mm_HandSolder" (id 2) (at 99.06 39.37 0)
@@
   (symbol (lib_id "Device:D_TVS") (at 74.93 43.18 90) (unit 1)
     (in_bom yes) (on_board yes) (fields_autoplaced)
-    (property "Reference" "D2" (id 0) (at 78.105 41.9099 90)
+    (property "Reference" "D5" (id 0) (at 78.105 41.9099 90)
       (effects (font (size 1.27 1.27)) (justify right))
     )
@@
   (symbol (lib_id "power:GND") (at 74.93 49.53 0) (unit 1)
     (in_bom yes) (on_board yes) (fields_autoplaced)
-    (property "Reference" "#PWR023" (id 0) (at 74.93 55.88 0)
+    (property "Reference" "#PWR027" (id 0) (at 74.93 55.88 0)
       (effects (font (size 1.27 1.27)) hide)
     )
@@
   (symbol (lib_id "power:+3V3") (at 104.14 32.385 0) (unit 1)
     (in_bom yes) (on_board yes) (fields_autoplaced)
-    (property "Reference" "#PWR024" (id 0) (at 104.14 36.195 0)
+    (property "Reference" "#PWR028" (id 0) (at 104.14 36.195 0)
       (effects (font (size 1.27 1.27)) hide)
     )
@@
   (symbol (lib_id "power:GND") (at 71.12 33.02 0) (unit 1)
     (in_bom yes) (on_board yes) (fields_autoplaced)
-    (property "Reference" "#PWR022" (id 0) (at 71.12 39.37 0)
+    (property "Reference" "#PWR026" (id 0) (at 71.12 39.37 0)
       (effects (font (size 1.27 1.27)) hide)
     )
@@
   (symbol (lib_id "Device:R_Small") (at 90.805 39.37 270) (unit 1)
     (in_bom yes) (on_board yes)
-    (property "Reference" "R4" (id 0) (at 90.805 41.91 90))
+    (property "Reference" "R7" (id 0) (at 90.805 41.91 90))
     (property "Value" "2k37" (id 1) (at 90.805 44.45 90))
     (property "Footprint" "Resistor_SMD:R_0603_1608Metric_Pad0.98x0.95mm_HandSolder" (id 2) (at 90.805 39.37 0)
@@
   (symbol (lib_id "Connector:TestPoint") (at 109.22 41.91 270) (unit 1)
     (in_bom yes) (on_board yes) (fields_autoplaced)
-    (property "Reference" "TP2" (id 0) (at 114.3 40.6399 90)
+    (property "Reference" "TP4" (id 0) (at 114.3 40.6399 90)
       (effects (font (size 1.27 1.27)) (justify left))
     )
@@
   (symbol (lib_id "Device:C_Small") (at 84.455 35.56 0) (unit 1)
     (in_bom yes) (on_board yes)
-    (property "Reference" "C11" (id 0) (at 73.66 34.29 0)
+    (property "Reference" "C12" (id 0) (at 73.66 34.29 0)
       (effects (font (size 1.27 1.27)) (justify left))
     )
@@
   (symbol (lib_id "Device:D_Small") (at 90.805 33.02 180) (unit 1)
     (in_bom yes) (on_board yes) (fields_autoplaced)
-    (property "Reference" "D3" (id 0) (at 90.805 26.67 0))
+    (property "Reference" "D6" (id 0) (at 90.805 26.67 0))
     (property "Value" "D_Small" (id 1) (at 90.805 29.21 0))
     (property "Footprint" "Diode_SMD:D_0603_1608Metric_Pad1.05x0.95mm_HandSolder" (id 2) (at 90.805 33.02 90)
@@
   (symbol (lib_id "power:GND") (at 109.22 43.18 0) (unit 1)
     (in_bom yes) (on_board yes) (fields_autoplaced)
-    (property "Reference" "#PWR025" (id 0) (at 109.22 49.53 0)
+    (property "Reference" "#PWR029" (id 0) (at 109.22 49.53 0)
       (effects (font (size 1.27 1.27)) hide)
     )
@@
   (symbol (lib_id "Device:R_Small") (at 104.14 36.83 0) (unit 1)
     (in_bom yes) (on_board yes) (fields_autoplaced)
-    (property "Reference" "R6" (id 0) (at 106.045 35.5599 0)
+    (property "Reference" "R9" (id 0) (at 106.045 35.5599 0)
       (effects (font (size 1.27 1.27)) (justify left))
     )
@@
   (symbol (lib_id "Device:D_Small") (at 99.06 33.02 180) (unit 1)
     (in_bom yes) (on_board yes) (fields_autoplaced)
-    (property "Reference" "D4" (id 0) (at 99.06 26.67 0))
+    (property "Reference" "D7" (id 0) (at 99.06 26.67 0))
     (property "Value" "D_Small" (id 1) (at 99.06 29.21 0))
     (property "Footprint" "Diode_SMD:D_0603_1608Metric_Pad1.05x0.95mm_HandSolder" (id 2) (at 99.06 33.02 90)

Commit message: Far better layout.
Parts:
- TP1: renamed from TP3; footprint TestPoint:TestPoint_THTPad_2.5x2.5mm_Drill1.2mm -> Library:Pogo Pin
- TP2: renamed from TP4; footprint TestPoint:TestPoint_THTPad_2.5x2.5mm_Drill1.2mm -> Library:Pogo Pin
- renumbered C12 to C11, D5 to D2, D6 to D3, D7 to D4, R7 to R4, R8 to R5, R9 to R6
Changed lines of the file:
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@@
   (symbol (lib_id "Device:R_Small") (at 99.06 39.37 270) (unit 1)
     (in_bom yes) (on_board yes)
-    (property "Reference" "R8" (id 0) (at 99.06 41.91 90))
+    (property "Reference" "R5" (id 0) (at 99.06 41.91 90))
     (property "Value" "2k37" (id 1) (at 99.06 44.45 90))
     (property "Footprint" "Resistor_SMD:R_0603_1608Metric_Pad0.98x0.95mm_HandSolder" (id 2) (at 99.06 39.37 0)
@@
   (symbol (lib_id "Device:D_TVS") (at 74.93 43.18 90) (unit 1)
     (in_bom yes) (on_board yes) (fields_autoplaced)
-    (property "Reference" "D5" (id 0) (at 78.105 41.9099 90)
+    (property "Reference" "D2" (id 0) (at 78.105 41.9099 90)
       (effects (font (size 1.27 1.27)) (justify right))
     )
@@
   (symbol (lib_id "power:GND") (at 74.93 49.53 0) (unit 1)
     (in_bom yes) (on_board yes) (fields_autoplaced)
-    (property "Reference" "#PWR027" (id 0) (at 74.93 55.88 0)
+    (property "Reference" "#PWR023" (id 0) (at 74.93 55.88 0)
       (effects (font (size 1.27 1.27)) hide)
     )
@@
   (symbol (lib_id "power:+3V3") (at 104.14 32.385 0) (unit 1)
     (in_bom yes) (on_board yes) (fields_autoplaced)
-    (property "Reference" "#PWR028" (id 0) (at 104.14 36.195 0)
+    (property "Reference" "#PWR024" (id 0) (at 104.14 36.195 0)
       (effects (font (size 1.27 1.27)) hide)
     )
@@
   (symbol (lib_id "power:GND") (at 71.12 33.02 0) (unit 1)
     (in_bom yes) (on_board yes) (fields_autoplaced)
-    (property "Reference" "#PWR026" (id 0) (at 71.12 39.37 0)
+    (property "Reference" "#PWR022" (id 0) (at 71.12 39.37 0)
       (effects (font (size 1.27 1.27)) hide)
     )
@@
   (symbol (lib_id "Device:R_Small") (at 90.805 39.37 270) (unit 1)
     (in_bom yes) (on_board yes)
-    (property "Reference" "R7" (id 0) (at 90.805 41.91 90))
+    (property "Reference" "R4" (id 0) (at 90.805 41.91 90))
     (property "Value" "2k37" (id 1) (at 90.805 44.45 90))
     (property "Footprint" "Resistor_SMD:R_0603_1608Metric_Pad0.98x0.95mm_HandSolder" (id 2) (at 90.805 39.37 0)
@@
   (symbol (lib_id "Connector:TestPoint") (at 109.22 41.91 270) (unit 1)
     (in_bom yes) (on_board yes) (fields_autoplaced)
-    (property "Reference" "TP4" (id 0) (at 114.3 40.6399 90)
+    (property "Reference" "TP2" (id 0) (at 114.3 40.6399 90)
       (effects (font (size 1.27 1.27)) (justify left))
     )
@@
       (effects (font (size 1.27 1.27)) (justify left) hide)
     )
-    (property "Footprint" "TestPoint:TestPoint_THTPad_2.5x2.5mm_Drill1.2mm" (id 2) (at 109.22 46.99 0)
+    (property "Footprint" "Library:Pogo Pin" (id 2) (at 109.22 46.99 0)
       (effects (font (size 1.27 1.27)) hide)
     )
@@
   (symbol (lib_id "Device:C_Small") (at 84.455 35.56 0) (unit 1)
     (in_bom yes) (on_board yes)
-    (property "Reference" "C12" (id 0) (at 73.66 34.29 0)
+    (property "Reference" "C11" (id 0) (at 73.66 34.29 0)
       (effects (font (size 1.27 1.27)) (justify left))
     )
@@
   (symbol (lib_id "Device:D_Small") (at 90.805 33.02 180) (unit 1)
     (in_bom yes) (on_board yes) (fields_autoplaced)
-    (property "Reference" "D6" (id 0) (at 90.805 26.67 0))
+    (property "Reference" "D3" (id 0) (at 90.805 26.67 0))
     (property "Value" "D_Small" (id 1) (at 90.805 29.21 0))
     (property "Footprint" "Diode_SMD:D_0603_1608Metric_Pad1.05x0.95mm_HandSolder" (id 2) (at 90.805 33.02 90)
@@
   (symbol (lib_id "power:GND") (at 109.22 43.18 0) (unit 1)
     (in_bom yes) (on_board yes) (fields_autoplaced)
-    (property "Reference" "#PWR029" (id 0) (at 109.22 49.53 0)
+    (property "Reference" "#PWR025" (id 0) (at 109.22 49.53 0)
       (effects (font (size 1.27 1.27)) hide)
     )
@@
   (symbol (lib_id "Device:R_Small") (at 104.14 36.83 0) (unit 1)
     (in_bom yes) (on_board yes) (fields_autoplaced)
-    (property "Reference" "R9" (id 0) (at 106.045 35.5599 0)
+    (property "Reference" "R6" (id 0) (at 106.045 35.5599 0)
       (effects (font (size 1.27 1.27)) (justify left))
     )
@@
   (symbol (lib_id "Device:D_Small") (at 99.06 33.02 180) (unit 1)
     (in_bom yes) (on_board yes) (fields_autoplaced)
-    (property "Reference" "D7" (id 0) (at 99.06 26.67 0))
+    (property "Reference" "D4" (id 0) (at 99.06 26.67 0))
     (property "Value" "D_Small" (id 1) (at 99.06 29.21 0))
     (property "Footprint" "Diode_SMD:D_0603_1608Metric_Pad1.05x0.95mm_HandSolder" (id 2) (at 99.06 33.02 90)
@@
   (symbol (lib_id "Connector:TestPoint") (at 109.22 39.37 270) (unit 1)
     (in_bom yes) (on_board yes) (fields_autoplaced)
-    (property "Reference" "TP3" (id 0) (at 114.3 38.0999 90)
+    (property "Reference" "TP1" (id 0) (at 114.3 38.0999 90)
       (effects (font (size 1.27 1.27)) (justify left))
     )
@@
       (effects (font (size 1.27 1.27)) (justify left) hide)
     )
-    (property "Footprint" "TestPoint:TestPoint_THTPad_2.5x2.5mm_Drill1.2mm" (id 2) (at 109.22 44.45 0)
+    (property "Footprint" "Library:Pogo Pin" (id 2) (at 109.22 44.45 0)
       (effects (font (size 1.27 1.27)) hide)
     )
